File: PedalBoard/PedalBoard.kicad_sch (KiCad schematic)
At the start: 9 parts, among them U1 YAAJ_BluePill_Part_Like, U4 MT3608

Commit message: згшщав
Changed lines of the file:
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@@
 	)
 	(sheet
-		(at 139.7 97.79)
+		(at 128.27 144.78)
 		(size 34.29 41.91)
 		(exclude_from_sim no)
@@
 		)
 		(property "Sheetname" "Preamp"
-			(at 139.7 97.0784 0)
+			(at 128.27 144.0684 0)
 			(effects
 				(font
@@
 		)
 		(property "Sheetfile" "preamp.kicad_sch"
-			(at 139.7 140.2846 0)
+			(at 128.27 187.2746 0)
 			(effects
 				(font
@@
 		)
 		(property "Field2" ""
-			(at 139.7 97.79 0)
+			(at 128.27 144.78 0)
 			(effects
 				(font
